File: EPROMShield/IOProtection.sch (KiCad schematic (older format))
At the start: 0 parts

Commit message: Finished schematic added caluclation for boost converter
Parts:
- added D? (x8): ZMMxx, Diode_SMD:D_MiniMELF, symbol Diode:ZMMxx
- added R? (x8): R, symbol Device:R
Connections:
- new net GND: D?.2 (A), D?.2 (A), D?.2 (A), D?.2 (A), D?.2 (A), D?.2 (A), D?.2 (A), D?.2 (A)
- new net Q0_IN: R?.1
- new net Q0_OUT: D?.1 (K), R?.2
- new net Q1_IN: R?.1
- new net Q1_OUT: D?.1 (K), R?.2
- new net Q2_IN: R?.1
- new net Q2_OUT: D?.1 (K), R?.2
- new net Q3_IN: R?.1
- new net Q3_OUT: D?.1 (K), R?.2
- new net Q4_IN: R?.1
- new net Q4_OUT: D?.1 (K), R?.2
- new net Q5_IN: R?.1
- new net Q5_OUT: D?.1 (K), R?.2
- new net Q6_IN: R?.1
- new net Q6_OUT: D?.1 (K), R?.2
- new net Q7_IN: R?.1
- new net Q7_OUT: D?.1 (K), R?.2
