File: EPROMShield/EPROMShield.kicad_pcb (KiCad board)
At the start: 2 copper layers, 101.6 x 53.3 mm, 13 parts, among them P1 Digital, P10 CONN_01X01, P11 CONN_01X01, P12 CONN_01X01, P13 CONN_01X01, P2 Power, P3 Analog, P4 Analog, P5 PWM, P6 PWM, P7 Communication, P8 CONN_01X01, P9 CONN_01X01

Commit message: Added netlist, fixed footprint L1
Parts:
- added C1: 1uF, Capacitor_THT:CP_Radial_D4.0mm_P1.50mm, F.Cu at (45.9, 114.1)
- added C2: 100n, Capacitor_SMD:C_0805_2012Metric_Pad1.18x1.45mm_HandSolder, F.Cu at (51.9, 112.8)
- added C3: 560pF, Capacitor_SMD:C_0805_2012Metric_Pad1.18x1.45mm_HandSolder, F.Cu at (63.3, 101.8)
- added C4: 50uF, Capacitor_THT:CP_Radial_D6.3mm_P2.50mm, F.Cu at (55.7, 100.8)
- added C5: 100n, Capacitor_SMD:C_0805_2012Metric_Pad1.18x1.45mm_HandSolder, F.Cu at (58.4, 106.2)
- added C6: 10uF, Capacitor_THT:CP_Radial_D6.3mm_P2.50mm, F.Cu at (38.7, 114.6)
- added C7: 1uF, Capacitor_THT:CP_Radial_D5.0mm_P2.50mm, F.Cu at (51.4, 108.0)
- added D1: LED_GN, LED_SMD:LED_1206_3216Metric_Pad1.42x1.75mm_HandSolder, F.Cu at (162.9, 22.8)
- added D10: ZMMxx, Diode_SMD:D_MiniMELF, F.Cu at (76.1, 22.7)
- added D11: ZMMxx, Diode_SMD:D_MiniMELF, F.Cu at (69.7, 22.7)
- added D12: ZMMxx, Diode_SMD:D_MiniMELF, F.Cu at (63.4, 22.7)
- added D13: ZMMxx, Diode_SMD:D_MiniMELF, F.Cu at (57.0, 22.7)
- added D14: ZMMxx, Diode_SMD:D_MiniMELF, F.Cu at (57.0, 26.0)
- added D15: BAS19, Package_TO_SOT_SMD:SOT-23, F.Cu at (70.3, 32.5)
- added D2: LED_RD, LED_SMD:LED_1206_3216Metric_Pad1.42x1.75mm_HandSolder, F.Cu at (162.9, 26.2)
- added D3: LED_BLUE, LED_SMD:LED_1206_3216Metric_Pad1.42x1.75mm_HandSolder, F.Cu at (63.9, 98.6)
- added D4: SK26ASMD, Diode_SMD:D_SMA_Handsoldering, F.Cu at (32.5, 107.7)
- added D5: 1N4001, Diode_THT:D_DO-41_SOD81_P10.16mm_Horizontal, F.Cu at (29.3, 103.3)
- added D6: 1N4001, Diode_THT:D_DO-41_SOD81_P10.16mm_Horizontal, F.Cu at (29.3, 99.0)
- added D7: ZMMxx, Diode_SMD:D_MiniMELF, F.Cu at (95.1, 22.7)
- added D8: ZMMxx, Diode_SMD:D_MiniMELF, F.Cu at (88.8, 22.7)
- added D9: ZMMxx, Diode_SMD:D_MiniMELF, F.Cu at (82.4, 22.7)
- added J1: Conn_02x16_Counter_Clockwise, Socket:DIP_Socket-32_W11.9_W12.7_W15.24_W17.78_W18.5_3M_232-1285-00-0602J, F.Cu at (175.9, 87.6)
- added L1: 100u, Inductor_SMD:L_Fastron_PISN_Handsoldering, F.Cu at (116.2, 106.1)
- added Q1: BC847, Package_TO_SOT_SMD:SOT-23, F.Cu at (61.3, 115.9)
- added Q2: BC847, Package_TO_SOT_SMD:SOT-23, F.Cu at (56.1, 48.2)
- added Q3: BSS83P, Package_TO_SOT_SMD:SOT-23, F.Cu at (100.5, 23.4)
- added Q4: BSS83P, Package_TO_SOT_SMD:SOT-23, F.Cu at (60.5, 48.2)
- added Q5: BSS83P, Package_TO_SOT_SMD:SOT-23, F.Cu at (60.8, 42.3)
- added Q6: BSS138, Package_TO_SOT_SMD:SOT-23, F.Cu at (70.3, 37.1)
- added Q7: BC847, Package_TO_SOT_SMD:SOT-23, F.Cu at (74.8, 32.5)
- added Q8: BC847, Package_TO_SOT_SMD:SOT-23, F.Cu at (56.1, 52.7)
- added R1: 470, Resistor_SMD:R_0805_2012Metric_Pad1.20x1.40mm_HandSolder, F.Cu at (168.2, 22.6)
- added R10: 1k, Resistor_SMD:R_0805_2012Metric_Pad1.20x1.40mm_HandSolder, F.Cu at (56.7, 115.7)
- added R11: 1k2, Resistor_SMD:R_0805_2012Metric_Pad1.20x1.40mm_HandSolder, F.Cu at (65.7, 35.6)
- added R12: 1k2, Resistor_SMD:R_0805_2012Metric_Pad1.20x1.40mm_HandSolder, F.Cu at (56.2, 44.4)
- added R13: 1k2, Resistor_SMD:R_0805_2012Metric_Pad1.20x1.40mm_HandSolder, F.Cu at (61.0, 38.5)
- added R14: 1k2, Resistor_SMD:R_0805_2012Metric_Pad1.20x1.40mm_HandSolder, F.Cu at (77.9, 25.8)
- added R15: 1k2, Resistor_SMD:R_0805_2012Metric_Pad1.20x1.40mm_HandSolder, F.Cu at (56.2, 41.5)
- added R16: 1k2, Resistor_SMD:R_0805_2012Metric_Pad1.20x1.40mm_HandSolder, F.Cu at (56.2, 38.5)
- added R17: 1k2, Resistor_SMD:R_0805_2012Metric_Pad1.20x1.40mm_HandSolder, F.Cu at (61.0, 35.6)
- added R18: 1k2, Resistor_SMD:R_0805_2012Metric_Pad1.20x1.40mm_HandSolder, F.Cu at (56.2, 35.6)
- added R19: 4k7, Resistor_SMD:R_0805_2012Metric_Pad1.20x1.40mm_HandSolder, F.Cu at (70.5, 28.8)
- added R2: 470, Resistor_SMD:R_0805_2012Metric_Pad1.20x1.40mm_HandSolder, F.Cu at (168.2, 25.5)
- added R20: 10k, Resistor_SMD:R_0805_2012Metric_Pad1.20x1.40mm_HandSolder, F.Cu at (65.7, 32.6)
- added R21: 15k, Resistor_SMD:R_0805_2012Metric_Pad1.20x1.40mm_HandSolder, F.Cu at (65.7, 29.7)
- added R22: 1k, Resistor_SMD:R_0805_2012Metric_Pad1.20x1.40mm_HandSolder, F.Cu at (61.0, 32.6)
- added R23: 1k5, Resistor_SMD:R_0805_2012Metric_Pad1.20x1.40mm_HandSolder, F.Cu at (29.8, 92.4)
- added R24: 10k, Resistor_SMD:R_0805_2012Metric_Pad1.20x1.40mm_HandSolder, F.Cu at (56.2, 32.6)
- added R25: 10k, Resistor_SMD:R_0805_2012Metric_Pad1.20x1.40mm_HandSolder, F.Cu at (61.0, 29.7)
- added R26: 1k, Resistor_SMD:R_0805_2012Metric_Pad1.20x1.40mm_HandSolder, F.Cu at (73.2, 25.8)
- added R27: 4k7, Resistor_SMD:R_0805_2012Metric_Pad1.20x1.40mm_HandSolder, F.Cu at (56.2, 29.7)
- added R28: 4k7, Resistor_SMD:R_0805_2012Metric_Pad1.20x1.40mm_HandSolder, F.Cu at (68.4, 25.8)
- added R3: 470, Resistor_SMD:R_0805_2012Metric_Pad1.20x1.40mm_HandSolder, F.Cu at (63.1, 106.2)
- added R4: 0.3, Resistor_SMD:R_1206_3216Metric_Pad1.30x1.75mm_HandSolder, F.Cu at (30.4, 118.0)
- added R5: 2k, Resistor_SMD:R_0805_2012Metric_Pad1.20x1.40mm_HandSolder, F.Cu at (51.8, 115.8)
- added R6: 180, Resistor_SMD:R_0805_2012Metric_Pad1.20x1.40mm_HandSolder, F.Cu at (56.7, 112.8)
- added R7: 18k4, Resistor_SMD:R_0805_2012Metric_Pad1.20x1.40mm_HandSolder, F.Cu at (63.1, 109.2)
- added R8: 3k, Resistor_SMD:R_0805_2012Metric_Pad1.20x1.40mm_HandSolder, F.Cu at (58.3, 109.2)
- added R9: 1k, Resistor_SMD:R_0805_2012Metric_Pad1.20x1.40mm_HandSolder, F.Cu at (61.4, 112.2)
- added TP1: TestPoint, TestPoint:TestPoint_Pad_D2.0mm, F.Cu at (65.8, 112.7)
- added TP2: TestPoint, TestPoint:TestPoint_Pad_D2.0mm, F.Cu at (82.3, 26.4)
- added TP3: TestPoint, TestPoint:TestPoint_Pad_D2.0mm, F.Cu at (65.1, 42.0)
- added U1: MC34063AD, Package_SO:SOIC-8_3.9x4.9mm_P1.27mm, F.Cu at (31.7, 113.2)
- added U2: LM317_TO-220, Package_TO_SOT_THT:TO-220-3_Vertical, F.Cu at (44.6, 100.8)
- added U3: 74AHC1GU04, Package_TO_SOT_SMD:SOT-353_SC-70-5_Handsoldering, F.Cu at (63.1, 26.3)
- moved P12 127.2 mm to (42.4, 91.9)
Connections:
- P1 pad 30: /27 -> /26
Other:
- net class Power added: clearance 0.2, trace_width 0.25, via_dia 0.6, via_drill 0.4
